File: _autosave-Snn-4layers.kicad_sch (KiCad schematic)
At the start: 77 parts, among them J1 Output connector, J2 Input connector, U1 ALD1106, U10 AP7366, U11 ADG619, U12 ADG619, U13 LTC6268xS8-10, U14 LT1715, U15 ADG619, U16 ADG619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

Commit message: semi final design
Parts:
- added C20: 100n, Capacitor_SMD:C_0402_1005Metric, symbol Device:C
Connections:
- net +5V: now also C20.2
- net GND: now also C20.1
Changed lines of the file:
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@@
     (stroke (width 0) (type default) (color 0 0 0 0))
   )
+  (wire (pts (xy 187.325 374.65) (xy 195.58 374.65))
+    (stroke (width 0) (type default) (color 0 0 0 0))
+  )
   (wire (pts (xy 183.515 34.925) (xy 179.07 34.925))
     (stroke (width 0) (type default) (color 0 0 0 0))
@@
     (stroke (width 0) (type default) (color 0 0 0 0))
   )
+  (wire (pts (xy 187.325 367.03) (xy 195.58 367.03))
+    (stroke (width 0) (type default) (color 0 0 0 0))
+  )
   (wire (pts (xy 337.82 124.46) (xy 353.06 124.46))
     (stroke (width 0) (type default) (color 0 0 0 0))
@@
     (pin "1")
   )
+  (symbol (lib_id "Device:C") (at 187.325 370.84 180) (unit 1)
+    (in_bom yes) (on_board yes) (fields_autoplaced)
+    (property "Reference" "C20" (id 0) (at 191.135 369.5699 0)
+      (effects (font (size 1.27 1.27)) (justify right))
+    )
+    (property "Value" "100n" (id 1) (at 191.135 372.1099 0)
+      (effects (font (size 1.27 1.27)) (justify right))
+    )
+    (property "Footprint" "Capacitor_SMD:C_0402_1005Metric" (id 2) (at 186.3598 367.03 0)
+      (effects (font (size 1.27 1.27)) hide)
+    )
+    (property "Datasheet" "~" (id 3) (at 187.325 370.84 0)
+      (effects (font (size 1.27 1.27)) hide)
+    )
+    (pin "1")
+    (pin "2")
+  )
   (symbol (lib_id "power:GND") (at 120.65 210.185 0) (unit 1)
     (in_bom yes) (on_board yes) (fields_autoplaced)
@@
       (reference "C19") (unit 1) (value "100n") (footprint "Capacitor_SMD:C_0402_1005Metric")
     )
+    (path "/12627b0b-2fa1-445a-8c51-b8dd4d94598a"
+      (reference "C20") (unit 1) (value "100n") (footprint "Capacitor_SMD:C_0402_1005Metric")
+    )
     (path "/95e3092a-6aa2-4d8b-8433-1f8b7e8ccd1b"
